File: int_out.kicad_pcb (KiCad board)
At the start: 2 copper layers, 85.3 x 100.1 mm, 73 parts, among them J1 Dimmers, J2 Relays, J3 switch inputs, J4 Inputs power 230V ac, J5 Power 230V ac, K1 HF49FD-005-1H11, K2 HF49FD-005-1H11, K3 HF49FD-005-1H11, K4 HF49FD-005-1H11, K5 HF49FD-005-1H11, K6 HF49FD-005-1H11, K7 HF49FD-005-1H11, K8 HF49FD-005-1H11, Q1 TIC226, Q2 TIC226, U1 H11AA1, U2 MOC3041M, U3 MOC3041M, U4 ESP32-WROOM-32UE, U5 LM1117-3.3, U6 TLP291-4, U7 ULN2803A, U8 TLP290-4

Commit message: bug fix in U5 (LM1117-3.3)
Parts:
- moved C7 4.50 mm to (147.4, 58.3), turned to 0 degrees
- moved C6 4.02 mm to (143.2, 58.3), turned to 180 degrees
- moved C9 1.03 mm to (151.4, 53.4), turned to 90 degrees
- moved U5 0.15 mm to (144.1, 52.5)
Connections:
- U5 pad 2: +5V -> +3V3
- U5 pad 3: +3V3 -> +5V
Routing:
- net +5V: track 61.3 -> 51.7 mm
- net +3V3: track 22.6 -> 20.1 mm
- net GND: track 134.7 -> 132.7 mm, vias 19 -> 20
