File: int_out.kicad_sch (KiCad schematic)
At the start: 75 parts, among them J1 Dimmers, J2 Relays, J3 switch inputs, J4 Inputs power 230V ac, J5 Power 230V ac, K1 HF49FD-005-1H11, K2 HF49FD-005-1H11, K3 HF49FD-005-1H11, K4 HF49FD-005-1H11, K5 HF49FD-005-1H11, K6 HF49FD-005-1H11, K7 HF49FD-005-1H11, K8 HF49FD-005-1H11, Q1 TIC226, Q2 TIC226, SW1 SWx4, U1 H11AA1, U2 MOC3041M, U3 MOC3041M, U4 ESP32-WROOM-32UE, U5 LM1117-3.3, U6 TLP291-4, U7 ULN2803A, U8 TLP290-4

Commit message: bug fix in U5 (LM1117-3.3)
Connections:
- net +3V3: now also U5.2 (VO); no longer U5.3 (VI)
- net +5V: now also U5.3 (VI); no longer U5.2 (VO)
Changed lines of the file:
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@@
-(kicad_sch (version 20230121) (generator eeschema)
+(kicad_sch (version 20230221) (generator eeschema)
   (paper "A4")
   (junction (at 182.88 108.585) (diameter 0) (color 0 0 0 0)
@@
     )
     (property "Footprint" "Relay_THT:Relay_HF49FDxxx-1h1" (at 59.69 110.49 0)
-      (effects (font (size 1.27 1.27)) (justify left) hide)
+      (effects (font (size 1.27 1.27)) (justify left))
     )
     (property "Datasheet" "" (at 50.8 109.22 0)
@@
     )
   )
-  (symbol (lib_id "Regulator_Linear:LM1117-3.3") (at 229.87 43.18 0) (unit 1)
-    (in_bom yes) (on_board yes) (dnp no) (fields_autoplaced)
-    (property "Reference" "U5" (at 229.87 37.3085 0)
-      (effects (font (size 1.27 1.27)))
-    )
-    (property "Value" "LM1117-3.3" (at 229.87 40.0836 0)
-      (effects (font (size 1.27 1.27)))
-    )
+  (symbol (lib_id "Regulator_Linear:LM1117-3.3") (at 229.87 43.18 0) (mirror y) (unit 1)
+    (in_bom yes) (on_board yes) (dnp no)
+    (property "Reference" "U5" (at 229.87 38.862 0)
+      (effects (font (size 1.27 1.27)))
+    )
+    (property "Value" "LM1117-3.3" (at 229.87 36.322 0)
+      (effects (font (size 1.27 1.27)))
+    )
